Commit message: add 3d-lidar test

File: orne_sim_description/urdf/orne_alpha.gazebo.xacro (robot description, xacro)
@@ -125,3 +125,8 @@
     </sensor>
   </gazebo>
+  <!-- VLP-16 specifications -->
+  <xacro:include filename="$(find orne_sim_description)/urdf/sensors/vlp16.urdf.xacro"/>
+    <xacro:vlp16_2d name="velodyne" parent="base_link">
+      <origin xyz="0.098 0.0 0.422" rpy="0 0 0"/>
+    </xacro:vlp16_2d>
 </robot>
