Commit message: add 3d lidar

File: orne_sim_description/urdf/orne_alpha.urdf.xacro (robot description, xacro)
@@ -26,7 +26,7 @@
       <origin xyz="0 0 0" rpy="0 0 0"/>
       <mass value="15.0"/>
-      <inertia ixx="1" ixy="0.0" ixz="0.0"
-               iyy="1" iyz="0.0"
-               izz="1" />
+      <inertia ixx="0.001" ixy="0.0" ixz="0.0"
+               iyy="0.001" iyz="0.0"
+               izz="0.001" />
     </inertial>
   </link>
@@ -54,7 +54,7 @@
       <origin xyz="0 0 0" />
       <mass value="0.2" />
-        <inertia ixx="0.1" ixy="0.0" ixz="0.0"
-                 iyy="0.1" iyz="0.0"
-                 izz="0.1" />
+        <inertia ixx="0.001" ixy="0.0" ixz="0.0"
+                 iyy="0.001" iyz="0.0"
+                 izz="0.001" />
     </inertial>
   </link>
@@ -82,7 +82,7 @@
         <origin xyz="0 0 0" />
         <mass value="0.2" />
-        <inertia ixx="0.1" ixy="0.0" ixz="0.0"
-                 iyy="0.1" iyz="0.0"
-                 izz="0.1" />
+        <inertia ixx="0.001" ixy="0.0" ixz="0.0"
+                 iyy="0.001" iyz="0.0"
+                 izz="0.001" />
       </inertial>
   </link>
@@ -134,3 +134,9 @@
     </inertial>
   </link>
+  <xacro:arg name="gpu" default="false"/>
+  <xacro:property name="gpu" value="$(arg gpu)" />
+  <xacro:include filename="$(find velodyne_description)/urdf/VLP-16.urdf.xacro"/>
+  <xacro:VLP-16 parent="base_scan" name="velodyne" topic="/velodyne_points" hz="10" samples="440" gpu="${gpu}">
+  <origin xyz="0 0 0.2" rpy="0 0 0" />
+  </xacro:VLP-16>
 </robot>

File: orne_sim_description/urdf/orne_box.urdf.xacro (robot description, xacro)
@@ -26,7 +26,7 @@
       <origin xyz="0 0 0" rpy="0 0 0"/>
       <mass value="15.0"/>
-      <inertia ixx="1" ixy="0.0" ixz="0.0"
-               iyy="1" iyz="0.0"
-               izz="1" />
+      <inertia ixx="0.001" ixy="0.0" ixz="0.0"
+               iyy="0.001" iyz="0.0"
+               izz="0.001" />
     </inertial>
   </link>
@@ -54,7 +54,7 @@
       <origin xyz="0 0 0" />
       <mass value="0.2" />
-        <inertia ixx="0.1" ixy="0.0" ixz="0.0"
-                 iyy="0.1" iyz="0.0"
-                 izz="0.1" />
+        <inertia ixx="0.001" ixy="0.0" ixz="0.0"
+                 iyy="0.001" iyz="0.0"
+                 izz="0.001" />
     </inertial>
   </link>
@@ -82,7 +82,7 @@
         <origin xyz="0 0 0" />
         <mass value="0.2" />
-        <inertia ixx="0.1" ixy="0.0" ixz="0.0"
-                 iyy="0.1" iyz="0.0"
-                 izz="0.1" />
+        <inertia ixx="0.001" ixy="0.0" ixz="0.0"
+                 iyy="0.001" iyz="0.0"
+                 izz="0.001" />
       </inertial>
   </link>

Commit message: change launch name

File: orne_sim_description/urdf/orne_alpha.urdf.xacro (robot description, xacro)
@@ -138,5 +138,5 @@
   <xacro:include filename="$(find velodyne_description)/urdf/VLP-16.urdf.xacro"/>
   <xacro:VLP-16 parent="base_scan" name="velodyne" topic="/velodyne_points" hz="10" samples="440" gpu="${gpu}">
-  <origin xyz="0 0 0.2" rpy="0 0 0" />
+  <origin xyz="-0.10 0 0.15" rpy="0 0 0" />
   </xacro:VLP-16>
 </robot>
